Commit message: Update

File: urdf/main.urdf.xacro (robot description, xacro)
@@ -48,4 +48,13 @@
 		xyz="0.03464101615 0.02 0"
 		rpy="1.570796326794896 0 -1.047197551196597"/>
+	<gazebo reference="rim_left">
+  		<material>Gazebo/Red</material>
+	</gazebo>
+	<gazebo reference="rim_back">
+  		<material>Gazebo/Green</material>
+	</gazebo>
+	<gazebo reference="rim_right">
+  		<material>Gazebo/Blue</material>
+	</gazebo>
 	<gazebo>
 		<plugin name="gazebo_ros_control" filename="libgazebo_ros_control.so">

File: urdf/rim.urdf.xacro (robot description, xacro)
@@ -90,8 +90,8 @@
 			<type>transmission_interface/SimpleTransmission</type>
 			<joint name="rim_${name}_joint">
-				<hardwareInterface>VelocityJointInterface</hardwareInterface>
+				<hardwareInterface>hardware_interface/VelocityJointInterface</hardwareInterface>
 			</joint>
 			<actuator name="rim_${name}_motor">
-				<hardwareInterface>VelocityJointInterface</hardwareInterface>
+				<hardwareInterface>hardware_interface/VelocityJointInterface</hardwareInterface>
 				<mechanicalReduction>1</mechanicalReduction>
 			</actuator>

Commit message: Update

File: urdf/main.urdf.xacro (robot description, xacro)
@@ -16,5 +16,5 @@
 	<visual>
 		<geometry>
-			<mesh filename="package://open_base/mesh/base.stl"/>
+			<mesh filename="package://omni3ros_pkg/mesh/base.stl"/>
 		</geometry>
 		<material name="base_material">
@@ -24,5 +24,5 @@
 	<collision>
 		<geometry>
-			<mesh filename="package://open_base/mesh/base.stl"/>
+			<mesh filename="package://omni3ros_pkg/mesh/base.stl"/>
 		</geometry>
 	</collision>
@@ -48,13 +48,4 @@
 		xyz="0.03464101615 0.02 0"
 		rpy="1.570796326794896 0 -1.047197551196597"/>
-	<gazebo reference="rim_left">
-  		<material>Gazebo/Red</material>
-	</gazebo>
-	<gazebo reference="rim_back">
-  		<material>Gazebo/Green</material>
-	</gazebo>
-	<gazebo reference="rim_right">
-  		<material>Gazebo/Blue</material>
-	</gazebo>
 	<gazebo>
 		<plugin name="gazebo_ros_control" filename="libgazebo_ros_control.so">

File: urdf/rim.urdf.xacro (robot description, xacro)
@@ -19,5 +19,5 @@
 			<visual>
 				<geometry>
-					<mesh filename="package://open_base/mesh/rim.stl"/>
+					<mesh filename="package://omni3ros_pkg/mesh/rim.stl"/>
 				</geometry>
 				<material name="rim_${name}_material">
@@ -27,5 +27,5 @@
 			<collision>
 				<geometry>
-					<mesh filename="package://open_base/mesh/rim.stl"/>
+					<mesh filename="package://omni3ros_pkg/mesh/rim.stl"/>
 				</geometry>
 			</collision>

File: urdf/roller.urdf.xacro (robot description, xacro)
@@ -17,5 +17,5 @@
 			<visual>
 				<geometry>
-					<mesh filename="package://open_base/mesh/roller.stl"/>
+					<mesh filename="package://omni3ros_pkg/mesh/roller.stl"/>
 				</geometry>
 				<material name="roller_material">
@@ -25,5 +25,5 @@
 			<collision>
 				<geometry>
-					<mesh filename="package://open_base/mesh/roller.stl"/>
+					<mesh filename="package://omni3ros_pkg/mesh/roller.stl"/>
 				</geometry>
 			</collision>

Commit message: Colors Added

File: urdf/main.urdf.xacro (robot description, xacro)
@@ -48,4 +48,16 @@
 		xyz="0.03464101615 0.02 0"
 		rpy="1.570796326794896 0 -1.047197551196597"/>
+	<gazebo reference="base_link">
+    		<material>Gazebo/White</material>
+  	</gazebo>
+	<gazebo reference="rim_left_link">
+    		<material>Gazebo/Red</material>
+  	</gazebo>
+	<gazebo reference="rim_back_link">
+    		<material>Gazebo/Green</material>
+  	</gazebo>
+	<gazebo reference="rim_right_link">
+    		<material>Gazebo/Blue</material>
+  	</gazebo>
 	<gazebo>
 		<plugin name="gazebo_ros_control" filename="libgazebo_ros_control.so">

File: urdf/roller.urdf.xacro (robot description, xacro)
@@ -29,4 +29,7 @@
 			</collision>
 		</link>
+	<gazebo reference="roller_${name}_rim_${parent}_link">
+    		<material>Gazebo/Black</material>
+  	</gazebo>
 		<joint name="roller_${name}_rim_${parent}_joint" type="continuous">
 			<parent link="rim_${parent}_link"/>
